File: KiCAD/Key_checker.kicad_pcb (KiCad board)
At the start: 2 copper layers, 67 x 68 mm, 18 parts, among them J1 Conn_01x03_Male, J2 Conn_01x03_Male, Q1 Q_Photo_NPN, SW1 SW_DIP_x01, U1 ESP32, U2 SSD1306

Commit message: Modified PCB
Parts:
- removed REF**: PinHeader_1x02_P2.54mm_Vertical, Connector_PinHeader_2.54mm:PinHeader_1x02_P2.54mm_Vertical
- added G***: LOGO, other:Keyicon, F.Cu at (172.7, 55.9)
- added J3: Conn_01x02_Male, Connector_PinHeader_2.54mm:PinHeader_1x02_P2.54mm_Horizontal, B.Cu at (203.2, 64.8)
- R1, R2, R3, R4: value R -> 470
- RV1: value R_POT -> 30k
- moved Q1 38.5 mm to (168.9, 26.7)
- moved SW1 13.5 mm to (166.4, 58.4)
- moved U2 12.5 mm to (200.7, 59.7), turned to 90 degrees
- moved J2 12.1 mm to (175.3, 33.0)
- moved RV1 5.08 mm to (215.9, 69.0)
- renumbered R5 to 10k1, R6 to 10k2, R7 to 10k3
Routing:
- net Net-(J2-Pad1): track 41.2 -> 0.00 mm
- net Net-(J2-Pad3): track 13.3 -> 31.2 mm
- net +3V3: track 69.4 -> 52.8 mm
- net +5V: track 49.6 -> 35.5 mm
- net Net-(J2-Pad2): track 20.4 -> 13.8 mm
- net Net-(10k3-Pad2): track 48.8 -> 46.4 mm
- net Net-(10k2-Pad2): track 57.4 -> 55.4 mm
- net GND: vias 1 -> 0
Other:
- outline, holes or cut-outs redrawn
- board text added: "3.3V"
- board text added: "External Connector"
- board text added: "Key Checker Rev1.1"
- board text added: "OLED Unit"
- board text added: "Photo Diode"
- board text added: "Power"
- board text added: "Put Keys!"
- board text added: "SCL"
- board text added: "SDA"
- board text added: "Sensor Adjust"
- board text added: "Status"
