File: KiCAD/Key_checker.sch (KiCad schematic (older format))
At the start: 14 parts, among them Q1 Q_Photo_NPN, SW1 SW_DIP_x01, U1 ESP32-Dev-Module-ESP32-footpr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, U2 SSD1306

Commit message: Key Checker's PCB is Completed!
Parts:
- added J1, J2: Conn_01x03_Male, Connector_PinHeader_2.54mm:PinHeader_1x03_P2.54mm_Horizontal, symbol Connector:Conn_01x03_Male
- U1: value ESP32-Dev-Module-ESP32-footprints-Shem-Lib -> ESP32
- U2: footprint Connector_PinHeader_1.27mm:PinHeader_1x04_P1.27mm_Vertical -> Connector_PinHeader_2.54mm:PinHeader_1x04_P2.54mm_Vertical
Connections:
- net GND: now also J1.1 (Pin_1); no longer Q1.2 (E), SW1.1
- net at RV1.2, U1.13 (IO12): now also J1.2 (Pin_2); no longer Q1.1 (C)
- net at R5.1, U1.6 (IO35): now also J1.3 (Pin_3); no longer SW1.2
- net +5V: now reaches R5.2, RV1.1, U1.19 (5V)
- net +3V3: now reaches R6.1, R7.1, U1.1 (3V3), U2.3 (VCC)
- new net: J2.2 (Pin_2), Q1.1 (C)
- new net: J2.1 (Pin_1), Q1.2 (E), SW1.1
- new net: J2.3 (Pin_3), SW1.2
Other:
- moved on the sheet: Q1, SW1
Changed lines of the file:
@@
 	6500 4100 6750 4100
-$Comp
-L Switch:SW_DIP_x01 SW1
-U 1 1 60D33FE5
-P 4000 3950
-F 0 "SW1" H 4000 4217 50  0000 C CNN
-F 1 "SW_DIP_x01" H 4000 4126 50  0000 C CNN
-F 2 "switch_micro:SS-10GL" H 4000 3950 50  0001 C CNN
-F 3 "~" H 4000 3950 50  0001 C CNN
-	1    4000 3950
-	0    -1   -1   0
-$EndComp
-$Comp
-L Device:Q_Photo_NPN Q1
-U 1 1 60D33560
-P 3000 4050
-F 0 "Q1" H 3190 4096 50  0000 L CNN
-F 1 "Q_Photo_NPN" H 3190 4005 50  0000 L CNN
-F 2 "LED_THT:LED_D5.0mm" H 3200 4150 50  0001 C CNN
-F 3 "~" H 3000 4050 50  0001 C CNN
-	1    3000 4050
-	1    0    0    -1
-$EndComp
 $Comp
 L Device:R R5
@@
 Wire Wire Line
 	4000 3500 4000 3650
-Connection ~ 4000 3650
-Wire Wire Line
-	4000 4450 4000 4250
-Wire Wire Line
-	3100 4250 3100 4450
 Wire Wire Line
 	3100 4450 3700 4450
-Connection ~ 4000 4450
-Wire Wire Line
-	4000 4450 4900 4450
-Wire Wire Line
-	4900 4350 3450 4350
-Wire Wire Line
-	3450 4350 3450 3850
-Wire Wire Line
-	3450 3850 3100 3850
-Wire Wire Line
-	3100 3850 3100 3450
-Connection ~ 3100 3850
+Wire Wire Line
+	4900 4350 3800 4350
 Wire Wire Line
 	4000 3200 4500 3200
@@
 	1    0    0    -1
 $EndComp
-Connection ~ 3100 4450
 $Comp
 L power:GND #PWR0102
@@
 $EndComp
 Wire Wire Line
-	2900 3450 3100 3450
-Wire Wire Line
 	2750 3300 2750 3200
 Wire Wire Line
@@
 F 0 "U2" H 4278 2313 50  0000 L CNN
 F 1 "SSD1306" H 4278 2222 50  0000 L CNN
-F 2 "Connector_PinHeader_1.27mm:PinHeader_1x04_P1.27mm_Vertical" H 4050 2550 50  0001 C CNN
+F 2 "Connector_PinHeader_2.54mm:PinHeader_1x04_P2.54mm_Vertical" H 4050 2550 50  0001 C CNN
 F 3 "" H 4050 2550 50  0001 C CNN
 	1    4050 2300
@@
 	3700 2900 3700 4450
 Connection ~ 3700 4450
-Wire Wire Line
-	3700 4450 4000 4450
 Wire Wire Line
 	4000 2500 4000 2700
@@
 P 5400 3050
 F 0 "U1" H 5400 3215 50  0000 C CNN
-F 1 "ESP32-Dev-Module-ESP32-footprints-Shem-Lib" H 5400 3124 50  0000 C CNN
+F 1 "ESP32" H 5400 3124 50  0000 C CNN
 F 2 "ESP32:DIP-38_1000_ELL" H 5400 3100 50  0001 C CNN
 F 3 "" H 5400 3100 50  0001 C CNN
@@
 	1    0    0    -1
 $EndComp
+$Comp
+L Switch:SW_DIP_x01 SW1
+U 1 1 60D33FE5
+P 1050 5100
+F 0 "SW1" H 1050 5367 50  0000 C CNN
+F 1 "SW_DIP_x01" H 1050 5276 50  0000 C CNN
+F 2 "switch_micro:SS-10GL" H 1050 5100 50  0001 C CNN
+F 3 "~" H 1050 5100 50  0001 C CNN
+	1    1050 5100
+	0    -1   -1   0
+$EndComp
+Connection ~ 4000 3650
+$Comp
+L Device:Q_Photo_NPN Q1
+U 1 1 60D33560
+P 950 4100
+F 0 "Q1" H 1140 4146 50  0000 L CNN
+F 1 "Q_Photo_NPN" H 1140 4055 50  0000 L CNN
+F 2 "LED_THT:LED_D5.0mm" H 1150 4200 50  0001 C CNN
+F 3 "~" H 950 4100 50  0001 C CNN
+	1    950  4100
+	1    0    0    -1
+$EndComp
+$Comp
+L Connector:Conn_01x03_Male J1
+U 1 1 60E05A12
+P 3800 5150
+F 0 "J1" V 3954 4962 50  0000 R CNN
+F 1 "Conn_01x03_Male" V 3863 4962 50  0000 R CNN
+F 2 "Connector_PinHeader_2.54mm:PinHeader_1x03_P2.54mm_Horizontal" H 3800 5150 50  0001 C CNN
+F 3 "~" H 3800 5150 50  0001 C CNN
+	1    3800 5150
+	0    -1   -1   0
+$EndComp
+$Comp
+L Connector:Conn_01x03_Male J2
+U 1 1 60E08B69
+P 1700 5650
+F 0 "J2" V 1854 5462 50  0000 R CNN
+F 1 "Conn_01x03_Male" V 1763 5462 50  0000 R CNN
+F 2 "Connector_PinHeader_2.54mm:PinHeader_1x03_P2.54mm_Horizontal" H 1700 5650 50  0001 C CNN
+F 3 "~" H 1700 5650 50  0001 C CNN
+	1    1700 5650
+	0    -1   -1   0
+$EndComp
+Wire Wire Line
+	3700 4950 3700 4450
+Wire Wire Line
+	3700 4450 4900 4450
+Wire Wire Line
+	3800 4950 3800 4350
+Connection ~ 3800 4350
+Wire Wire Line
+	3900 3650 4000 3650
+Wire Wire Line
+	3800 3450 3800 4350
+Wire Wire Line
+	2900 3450 3800 3450
+Wire Wire Line
+	3900 3650 3900 4950
+Wire Wire Line
+	1600 5450 1600 5400
+Wire Wire Line
+	1600 5400 1050 5400
+Wire Wire Line
+	1600 5400 1600 4300
+Wire Wire Line
+	1600 4300 1050 4300
+Connection ~ 1600 5400
+Wire Wire Line
+	1050 4800 1800 4800
+Wire Wire Line
+	1800 4800 1800 5450
+Wire Wire Line
+	1700 5450 1700 3900
+Wire Wire Line
+	1700 3900 1050 3900
+$Comp
+L power:+5V #PWR0105
+U 1 1 60E1FADC
+P 2750 3200
+F 0 "#PWR0105" H 2750 3050 50  0001 C CNN
+F 1 "+5V" H 2765 3373 50  0000 C CNN
+F 2 "" H 2750 3200 50  0001 C CNN
+F 3 "" H 2750 3200 50  0001 C CNN
+	1    2750 3200
+	1    0    0    -1
+$EndComp
+Connection ~ 2750 3200
+$Comp
+L power:+3V3 #PWR0106
+U 1 1 60E20281
+P 3300 3150
+F 0 "#PWR0106" H 3300 3000 50  0001 C CNN
+F 1 "+3V3" H 3315 3323 50  0000 C CNN
+F 2 "" H 3300 3150 50  0001 C CNN
+F 3 "" H 3300 3150 50  0001 C CNN
+	1    3300 3150
+	1    0    0    -1
+$EndComp
+Wire Wire Line
+	3300 3150 4100 3150
+Connection ~ 4100 3150
 $EndSCHEMATC

Commit message: Fixed problem in PCB
Parts:
- R1, R2, R3, R4: value R -> 470
- RV1: value R_POT -> 30k
- renumbered R5 to 10k, R6 to 10k, R7 to 10k
Changed lines of the file:
@@
 P 6900 4100
 F 0 "R1" H 6970 4146 50  0000 L CNN
-F 1 "R" H 6970 4055 50  0000 L CNN
+F 1 "470" H 6970 4055 50  0000 L CNN
 F 2 "Resistor_SMD:R_0603_1608Metric_Pad0.98x0.95mm_HandSolder" V 6830 4100 50  0001 C CNN
 F 3 "~" H 6900 4100 50  0001 C CNN
@@
 P 6400 4550
 F 0 "R2" H 6470 4596 50  0000 L CNN
-F 1 "R" H 6470 4505 50  0000 L CNN
+F 1 "470" H 6470 4505 50  0000 L CNN
 F 2 "Resistor_SMD:R_0603_1608Metric_Pad0.98x0.95mm_HandSolder" V 6330 4550 50  0001 C CNN
 F 3 "~" H 6400 4550 50  0001 C CNN
@@
 P 6400 5050
 F 0 "R3" H 6470 5096 50  0000 L CNN
-F 1 "R" H 6470 5005 50  0000 L CNN
+F 1 "470" H 6470 5005 50  0000 L CNN
 F 2 "Resistor_SMD:R_0603_1608Metric_Pad0.98x0.95mm_HandSolder" V 6330 5050 50  0001 C CNN
 F 3 "~" H 6400 5050 50  0001 C CNN
@@
 P 6400 4800
 F 0 "R4" H 6470 4846 50  0000 L CNN
-F 1 "R" H 6470 4755 50  0000 L CNN
+F 1 "470" H 6470 4755 50  0000 L CNN
 F 2 "Resistor_SMD:R_0603_1608Metric_Pad0.98x0.95mm_HandSolder" V 6330 4800 50  0001 C CNN
 F 3 "~" H 6400 4800 50  0001 C CNN
@@
 	6500 4100 6750 4100
 $Comp
-L Device:R R5
+L Device:R 10k
 U 1 1 60D7AB9A
 P 4000 3350
-F 0 "R5" H 4070 3396 50  0000 L CNN
+F 0 "10k" H 4070 3396 50  0000 L CNN
 F 1 "R" H 4070 3305 50  0000 L CNN
 F 2 "Resistor_SMD:R_0603_1608Metric_Pad0.98x0.95mm_HandSolder" V 3930 3350 50  0001 C CNN
@@
 P 2750 3450
 F 0 "RV1" H 2681 3496 50  0000 R CNN
-F 1 "R_POT" H 2681 3405 50  0000 R CNN
+F 1 "30k" H 2681 3405 50  0000 R CNN
 F 2 "Potentiometer_THT:Potentiometer_ACP_CA6-H2,5_Horizontal" H 2750 3450 50  0001 C CNN
 F 3 "~" H 2750 3450 50  0001 C CNN
@@
 	3900 2800 3900 2500
 $Comp
-L Device:R R6
+L Device:R 10k
 U 1 1 60DD395E
 P 4300 3000
-F 0 "R6" H 4370 3046 50  0000 L CNN
+F 0 "10k" H 4370 3046 50  0000 L CNN
 F 1 "R" H 4370 2955 50  0000 L CNN
 F 2 "Resistor_SMD:R_0603_1608Metric_Pad0.98x0.95mm_HandSolder" V 4230 3000 50  0001 C CNN
@@
 $EndComp
 $Comp
-L Device:R R7
+L Device:R 10k
 U 1 1 60DD4749
 P 4600 3000
-F 0 "R7" H 4670 3046 50  0000 L CNN
+F 0 "10k" H 4670 3046 50  0000 L CNN
 F 1 "R" H 4670 2955 50  0000 L CNN
 F 2 "Resistor_SMD:R_0603_1608Metric_Pad0.98x0.95mm_HandSolder" V 4530 3000 50  0001 C CNN

Commit message: Modified PCB
Parts:
- added J3: Conn_01x02_Male, Connector_PinHeader_2.54mm:PinHeader_1x02_P2.54mm_Horizontal, symbol Connector:Conn_01x02_Male
- renumbered 10k to 10k1, 10k to 10k2, 10k to 10k3
Connections:
- net +5V: now also J3.1 (Pin_1)
- net GND: now also J3.2 (Pin_2)
Changed lines of the file:
@@
 	6500 4100 6750 4100
 $Comp
-L Device:R 10k
+L Device:R 10k1
 U 1 1 60D7AB9A
 P 4000 3350
-F 0 "10k" H 4070 3396 50  0000 L CNN
+F 0 "10k1" H 4070 3396 50  0000 L CNN
 F 1 "R" H 4070 3305 50  0000 L CNN
 F 2 "Resistor_SMD:R_0603_1608Metric_Pad0.98x0.95mm_HandSolder" V 3930 3350 50  0001 C CNN
@@
 	3900 2800 3900 2500
 $Comp
-L Device:R 10k
+L Device:R 10k2
 U 1 1 60DD395E
 P 4300 3000
-F 0 "10k" H 4370 3046 50  0000 L CNN
+F 0 "10k2" H 4370 3046 50  0000 L CNN
 F 1 "R" H 4370 2955 50  0000 L CNN
 F 2 "Resistor_SMD:R_0603_1608Metric_Pad0.98x0.95mm_HandSolder" V 4230 3000 50  0001 C CNN
@@
 $EndComp
 $Comp
-L Device:R 10k
+L Device:R 10k3
 U 1 1 60DD4749
 P 4600 3000
-F 0 "10k" H 4670 3046 50  0000 L CNN
+F 0 "10k3" H 4670 3046 50  0000 L CNN
 F 1 "R" H 4670 2955 50  0000 L CNN
 F 2 "Resistor_SMD:R_0603_1608Metric_Pad0.98x0.95mm_HandSolder" V 4530 3000 50  0001 C CNN
@@
 	3300 3150 4100 3150
 Connection ~ 4100 3150
+$Comp
+L power:+5V #PWR0107
+U 1 1 61BC6DC6
+P 2600 1600
+F 0 "#PWR0107" H 2600 1450 50  0001 C CNN
+F 1 "+5V" H 2615 1773 50  0000 C CNN
+F 2 "" H 2600 1600 50  0001 C CNN
+F 3 "" H 2600 1600 50  0001 C CNN
+	1    2600 1600
+	1    0    0    -1
+$EndComp
+$Comp
+L power:GND #PWR0108
+U 1 1 61BC750F
+P 2600 1700
+F 0 "#PWR0108" H 2600 1450 50  0001 C CNN
+F 1 "GND" H 2605 1527 50  0000 C CNN
+F 2 "" H 2600 1700 50  0001 C CNN
+F 3 "" H 2600 1700 50  0001 C CNN
+	1    2600 1700
+	1    0    0    -1
+$EndComp
+$Comp
+L Connector:Conn_01x02_Male J3
+U 1 1 61BC53FB
+P 2400 1600
+F 0 "J3" H 2508 1781 50  0000 C CNN
+F 1 "Conn_01x02_Male" H 2508 1690 50  0000 C CNN
+F 2 "Connector_PinHeader_2.54mm:PinHeader_1x02_P2.54mm_Horizontal" H 2400 1600 50  0001 C CNN
+F 3 "~" H 2400 1600 50  0001 C CNN
+	1    2400 1600
+	1    0    0    -1
+$EndComp
 $EndSCHEMATC
